Commit message: Add rv7fr_dh_floor_gazebo moveit config to test Gazebo-Moveit

File: melfa_description/urdf/rv7fr-dh-floor-gazebo.urdf (robot description, URDF)
Before this commit: robot rv7fr, 10 links, 9 joints
Links:
- link base: mass None -> 17.73185816
- link floor: mass None -> 17.73185816
- link link1: mass None -> 8.1786898
- link link2: mass None -> 12.68401416
- link link3: mass None -> 5.21740642
- link link4: mass None -> 3.8290545
- link link5: mass None -> 0.79715023
- link link6: mass None -> 0.0253625682818
Joints:
- joint joint1: limit lower=${RADIANS*(-240.)} upper=${RADIANS*(240.)} effort=119.36611817 velocity=${RADIANS*(360.)} -> lower=-4.18879020533 upper=4.18879020533 effort=119.36611817 velocity=6.283185308
- joint joint2: limit lower=${RADIANS*(-107.-90.)} upper=${RADIANS*(125.-90.)} effort=107.16168698 velocity=${RADIANS*(401.)} -> lower=-3.43829862688 upper=0.610865238278 effort=107.16168698 velocity=6.99877030141; origin xyz=0. 0. 0.175 rpy=${RADIANS*(-90.)} 0.0 0.0 -> xyz=0. 0. 0.175 rpy=-1.570796327 0.0 0.0
- joint joint3: limit lower=${RADIANS*(-90.)} upper=${RADIANS*(156.-90.)} effort=50.92959239 velocity=${RADIANS*(450.)} -> lower=-1.570796327 upper=1.15191730647 effort=50.92959239 velocity=7.853981635
- joint joint4: limit lower=${RADIANS*(-200.)} upper=${RADIANS*(200.)} effort=16.2 velocity=${RADIANS*(337.)} -> lower=-3.49065850444 upper=3.49065850444 effort=16.2 velocity=5.88175957999; origin xyz=0.05 0 0 rpy=${RADIANS*(-90.)} 0 0 -> xyz=0.05 0 0 rpy=-1.570796327 0 0
- joint joint5: limit lower=${RADIANS*(-120.)} upper=${RADIANS*(120.)} effort=16.2 velocity=${RADIANS*(450.)} -> lower=-2.09439510267 upper=2.09439510267 effort=16.2 velocity=7.853981635; origin xyz=0 0 ${0.2745+0.095} rpy=${RADIANS*(90.)} 0 0 -> xyz=0 0 0.3695 rpy=1.570796327 0 0
- joint joint6: limit lower=${RADIANS*(-360.)} upper=${RADIANS*(360.)} effort=6.86 velocity=${RADIANS*(720.)} -> lower=-6.283185308 upper=6.283185308 effort=6.86 velocity=12.566370616; origin xyz=0 0 0 rpy=${RADIANS*(-90.)} 0 0 -> xyz=0 0 0 rpy=-1.570796327 0 0

File: melfa_description/urdf/rv7fr-dh-floor-gazebo.urdf.xacro (robot description, xacro)
@@ -296,9 +296,9 @@
     <axis xyz="0 0 0"/>
   </joint>
-  <!--gazebo>
+  <gazebo>
     <plugin name="gazebo_ros_control" filename="libgazebo_ros_control.so">
       <robotNamespace>/rv7fr</robotNamespace>
       <robotSimType>gazebo_ros_control/DefaultRobotHWSim</robotSimType>
     </plugin>
-  </gazebo-->
+  </gazebo>
 </robot>

File: melfa_description/urdf/rv7fr-dh-floor-gazebo2.urdf (robot description, URDF)
Before this commit: robot rv7fr, 10 links, 9 joints
Links:
- link base: mass None -> 17.73185816
- link floor: mass None -> 17.73185816
- link link1: mass None -> 8.1786898
- link link2: mass None -> 12.68401416
- link link3: mass None -> 5.21740642
- link link4: mass None -> 3.8290545
- link link5: mass None -> 0.79715023
- link link6: mass None -> 0.0253625682818
Joints:
- joint joint1: limit lower=${RADIANS*(-240.)} upper=${RADIANS*(240.)} effort=119.36611817 velocity=${RADIANS*(360.)} -> lower=-4.18879020533 upper=4.18879020533 effort=119.36611817 velocity=6.283185308
- joint joint2: limit lower=${RADIANS*(-107.-90.)} upper=${RADIANS*(125.-90.)} effort=107.16168698 velocity=${RADIANS*(401.)} -> lower=-3.43829862688 upper=0.610865238278 effort=107.16168698 velocity=6.99877030141; origin xyz=0. 0. 0.175 rpy=${RADIANS*(-90.)} 0.0 0.0 -> xyz=0. 0. 0.175 rpy=-1.570796327 0.0 0.0
- joint joint3: limit lower=${RADIANS*(-90.)} upper=${RADIANS*(156.-90.)} effort=50.92959239 velocity=${RADIANS*(450.)} -> lower=-1.570796327 upper=1.15191730647 effort=50.92959239 velocity=7.853981635
- joint joint4: limit lower=${RADIANS*(-200.)} upper=${RADIANS*(200.)} effort=16.2 velocity=${RADIANS*(337.)} -> lower=-3.49065850444 upper=3.49065850444 effort=16.2 velocity=5.88175957999; origin xyz=0.05 0 0 rpy=${RADIANS*(-90.)} 0 0 -> xyz=0.05 0 0 rpy=-1.570796327 0 0
- joint joint5: limit lower=${RADIANS*(-120.)} upper=${RADIANS*(120.)} effort=16.2 velocity=${RADIANS*(450.)} -> lower=-2.09439510267 upper=2.09439510267 effort=16.2 velocity=7.853981635; origin xyz=0 0 ${0.2745+0.095} rpy=${RADIANS*(90.)} 0 0 -> xyz=0 0 0.3695 rpy=1.570796327 0 0
- joint joint6: limit lower=${RADIANS*(-360.)} upper=${RADIANS*(360.)} effort=6.86 velocity=${RADIANS*(720.)} -> lower=-6.283185308 upper=6.283185308 effort=6.86 velocity=12.566370616; origin xyz=0 0 0 rpy=${RADIANS*(-90.)} 0 0 -> xyz=0 0 0 rpy=-1.570796327 0 0

File: melfa_description/urdf/rv7fr-dh-floor.urdf (robot description, URDF)
Before this commit: robot rv7fr, 10 links, 9 joints
Links:
- link base: mass None -> 17.73185816
- link floor: mass None -> 17.73185816
- link link1: mass None -> 8.1786898
- link link2: mass None -> 12.68401416
- link link3: mass None -> 5.21740642
- link link4: mass None -> 3.8290545
- link link5: mass None -> 0.79715023
- link link6: mass None -> 0.0253625682818
Joints:
- joint joint1: limit lower=${RADIANS*(-240.)} upper=${RADIANS*(240.)} effort=119.36611817 velocity=${RADIANS*(360.)} -> lower=-4.18879020533 upper=4.18879020533 effort=119.36611817 velocity=6.283185308
- joint joint2: limit lower=${RADIANS*(-107.-90.)} upper=${RADIANS*(125.-90.)} effort=107.16168698 velocity=${RADIANS*(401.)} -> lower=-3.43829862688 upper=0.610865238278 effort=107.16168698 velocity=6.99877030141; origin xyz=0. 0. 0.175 rpy=${RADIANS*(-90.)} 0.0 0.0 -> xyz=0. 0. 0.175 rpy=-1.570796327 0.0 0.0
- joint joint3: limit lower=${RADIANS*(-90.)} upper=${RADIANS*(156.-90.)} effort=50.92959239 velocity=${RADIANS*(450.)} -> lower=-1.570796327 upper=1.15191730647 effort=50.92959239 velocity=7.853981635
- joint joint4: limit lower=${RADIANS*(-200.)} upper=${RADIANS*(200.)} effort=16.2 velocity=${RADIANS*(337.)} -> lower=-3.49065850444 upper=3.49065850444 effort=16.2 velocity=5.88175957999; origin xyz=0.05 0 0 rpy=${RADIANS*(-90.)} 0 0 -> xyz=0.05 0 0 rpy=-1.570796327 0 0
- joint joint5: limit lower=${RADIANS*(-120.)} upper=${RADIANS*(120.)} effort=16.2 velocity=${RADIANS*(450.)} -> lower=-2.09439510267 upper=2.09439510267 effort=16.2 velocity=7.853981635; origin xyz=0 0 ${0.2745+0.095} rpy=${RADIANS*(90.)} 0 0 -> xyz=0 0 0.3695 rpy=1.570796327 0 0
- joint joint6: limit lower=${RADIANS*(-360.)} upper=${RADIANS*(360.)} effort=6.86 velocity=${RADIANS*(720.)} -> lower=-6.283185308 upper=6.283185308 effort=6.86 velocity=12.566370616; origin xyz=0 0 0 rpy=${RADIANS*(-90.)} 0 0 -> xyz=0 0 0 rpy=-1.570796327 0 0

File: melfa_description/urdf/temp.urdf (robot description, URDF)
Before this commit: robot rv7fr, 10 links, 9 joints
Links:
- link base: mass None -> 17.73185816
- link floor: mass None -> 17.73185816
- link link1: mass None -> 8.1786898
- link link2: mass None -> 12.68401416
- link link3: mass None -> 5.21740642
- link link4: mass None -> 3.8290545
- link link5: mass None -> 0.79715023
- link link6: mass None -> 0.0253625682818
Joints:
- joint joint1: limit lower=${RADIANS*(-240.)} upper=${RADIANS*(240.)} effort=119.36611817 velocity=${RADIANS*(360.)} -> lower=-4.18879020533 upper=4.18879020533 effort=119.36611817 velocity=6.283185308
- joint joint2: limit lower=${RADIANS*(-107.-90.)} upper=${RADIANS*(125.-90.)} effort=107.16168698 velocity=${RADIANS*(401.)} -> lower=-3.43829862688 upper=0.610865238278 effort=107.16168698 velocity=6.99877030141; origin xyz=0. 0. 0.175 rpy=${RADIANS*(-90.)} 0.0 0.0 -> xyz=0. 0. 0.175 rpy=-1.570796327 0.0 0.0
- joint joint3: limit lower=${RADIANS*(-90.)} upper=${RADIANS*(156.-90.)} effort=50.92959239 velocity=${RADIANS*(450.)} -> lower=-1.570796327 upper=1.15191730647 effort=50.92959239 velocity=7.853981635
- joint joint4: limit lower=${RADIANS*(-200.)} upper=${RADIANS*(200.)} effort=16.2 velocity=${RADIANS*(337.)} -> lower=-3.49065850444 upper=3.49065850444 effort=16.2 velocity=5.88175957999; origin xyz=0.05 0 0 rpy=${RADIANS*(-90.)} 0 0 -> xyz=0.05 0 0 rpy=-1.570796327 0 0
- joint joint5: limit lower=${RADIANS*(-120.)} upper=${RADIANS*(120.)} effort=16.2 velocity=${RADIANS*(450.)} -> lower=-2.09439510267 upper=2.09439510267 effort=16.2 velocity=7.853981635; origin xyz=0 0 ${0.2745+0.095} rpy=${RADIANS*(90.)} 0 0 -> xyz=0 0 0.3695 rpy=1.570796327 0 0
- joint joint6: limit lower=${RADIANS*(-360.)} upper=${RADIANS*(360.)} effort=6.86 velocity=${RADIANS*(720.)} -> lower=-6.283185308 upper=6.283185308 effort=6.86 velocity=12.566370616; origin xyz=0 0 0 rpy=${RADIANS*(-90.)} 0 0 -> xyz=0 0 0 rpy=-1.570796327 0 0
