Commit message: Pose marker class added for interactive programmable start goal state

File: melfa_description/urdf/rv7fr-dh-zero-table-sensor.urdf (robot description, URDF)
Before this commit: robot rv7fr, 12 links, 11 joints
Links:
- link base: mass None -> 17.73185816
- link link1: mass None -> 8.1786898
- link link2: mass None -> 12.68401416
- link link3: mass None -> 5.21740642
- link link4: mass None -> 3.8290545
- link link5: mass None -> 0.79715023
- link link6: mass None -> 0.0253625682818
Joints:
- joint joint1: limit lower=${radians(-240)} upper=${radians(240)} effort=119.36611817 velocity=${radians(360)} -> lower=-4.18879020479 upper=4.18879020479 effort=119.36611817 velocity=6.28318530718
- joint joint2: limit lower=${radians(-107)} upper=${radians(125)} effort=107.16168698 velocity=${radians(401)} -> lower=-1.86750229963 upper=2.18166156499 effort=107.16168698 velocity=6.9987703005; origin xyz=0 0 0.175 rpy=${radians(-90)} ${radians(-90)} 0.0 -> xyz=0 0 0.175 rpy=-1.57079632679 -1.57079632679 0.0
- joint joint3: limit lower=${radians(0)} upper=${radians(156)} effort=50.92959239 velocity=${radians(450)} -> lower=0.0 upper=2.72271363311 effort=50.92959239 velocity=7.85398163397; origin xyz=0.34 0 0 rpy=0 0 ${radians(-90)} -> xyz=0.34 0 0 rpy=0 0 -1.57079632679
- joint joint4: limit lower=${radians(-200)} upper=${radians(200)} effort=16.2 velocity=${radians(337)} -> lower=-3.49065850399 upper=3.49065850399 effort=16.2 velocity=5.88175957922; origin xyz=0.05 0 0 rpy=${radians(-90)} 0 0 -> xyz=0.05 0 0 rpy=-1.57079632679 0 0
- joint joint5: limit lower=${radians(-120)} upper=${radians(120)} effort=16.2 velocity=${radians(450)} -> lower=-2.09439510239 upper=2.09439510239 effort=16.2 velocity=7.85398163397; origin xyz=0 0 ${0.2745+0.095} rpy=${radians(90)} 0 0 -> xyz=0 0 0.3695 rpy=1.57079632679 0 0
- joint joint6: limit lower=${radians(-360)} upper=${radians(360)} effort=6.86 velocity=${radians(720)} -> lower=-6.28318530718 upper=6.28318530718 effort=6.86 velocity=12.5663706144; origin xyz=0 0 0 rpy=${radians(-90)} 0 0 -> xyz=0 0 0 rpy=-1.57079632679 0 0
- joint realsense_sensor1: origin xyz=0 0 0 rpy=0 ${radians(-90)} 0 -> xyz=0 0 0 rpy=0 -1.57079632679 0
- joint realsense_sensor2: origin xyz=0 0 0 rpy=${radians(-90)} 0 ${radians(-90)} -> xyz=0 0 0 rpy=-1.57079632679 0 -1.57079632679
